File: templates/f135d3a.kicad_sch (KiCad schematic)
At the start: 1 part

Commit message: KiSchEdit train of thought totaly changed. Now directly imagining for layout
Parts:
- {{schEditModule.symEditSym.sym.designator}}1: renamed from {{schEditSym.symEditSym.sym.designator}}1; symbol {{schEditSym.libName}}:{{schEditSym.symEditSym.sym.name}} -> {{schEditModule.libName}}:{{schEditModule.symEditSym.sym.name}}
Changed lines of the file:
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@@
 	(generator_version "8.0")
 	(paper "A4")
-{% for schEditSym in schEditSyms %} {# KiSchEditSym type #}
+{% for schEditModule in schEditModules %} {# KiSchEditSym type #}
 	(symbol
-		(lib_id "{{schEditSym.libName}}:{{schEditSym.symEditSym.sym.name}}")
-		(at 12.7 15.24 0)
+		(lib_id "{{schEditModule.libName}}:{{schEditModule.symEditSym.sym.name}}")
+		(at {{schEditModule.symx}} {{schEditModule.symy}} 0)
 		(unit 1)
 		(exclude_from_sim no)
@@
 		(dnp no)
 		(fields_autoplaced yes)
-		(property "Reference" "{{schEditSym.symEditSym.sym.designator}}1"
-			(at 28.194 13.97 0)
+		(property "Reference" "{{schEditModule.symEditSym.sym.designator}}1"
+			(at {{schEditModule.symx}} {{schEditModule.symy}} 0)
 			(effects
 				(font
@@
 			(project ""
 				(path "/97f17985-da40-43fd-b268-8c96b481a2af"
-					(reference "{{schEditSym.symEditSym.sym.designator}}1")
+					(reference "{{schEditModule.symEditSym.sym.designator}}1")
 					(unit 1)
 				)
@@
 		)
 	)
-{% endfor %}{# schEditSyms #}
+{% endfor %}{# schEditModules #}
 	(sheet_instances
 		(path "/"
