File: templates/v8/f135d3a.kicad_sch (KiCad schematic)
At the start: 1 part

Commit message: 13-add-ability-to-show-pin-number:ability to show pin numbers
Connections:
- net {{schEditNode.name}}: now also {{schEditModule.symEditSym.sym.designator}}1.{{symEditPin.pin.number}} ({{symEditPin.pin.name}}); no longer {{schEditModule.symEditSym.sym.designator}}1. ({{symEditPin.pin.name}})

Commit message: 14-add-leftright-to-choose-location-of-the-pins: now position of the pin is not tied to shape of the pin so I can put bidirectional pin also directional pin added to two.csv
Changed lines of the file:
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@@
 	(paper "User" {{pageWidth}} {{pageHeight}})
 {% for schEditModule in schEditModules %} {# _KiSchEditModule type #}
-{% 		if not schEditModule.numOfSchEditConns["input"] == 0 %}
-{% 			for schEditWire in schEditModule.schEditWireCont["input"].wires %}
+{% 		if not schEditModule.numOfSchEditConns["left"] == 0 %}
+{% 			for schEditWire in schEditModule.schEditWireCont["left"].wires %}
 {% 				if loggingEnabled == True %}
 	{{schEditWire.name}}
@@
 {% endfor %}{# schEditModules #}
 {% for schEditModule in schEditModules %} {# _KiSchEditModule type #}
-{% 		if not schEditModule.numOfSchEditConns["output"] == 0 %}
-{% 			for schEditWire in schEditModule.schEditWireCont["output"].wires %}
+{% 		if not schEditModule.numOfSchEditConns["right"] == 0 %}
+{% 			for schEditWire in schEditModule.schEditWireCont["right"].wires %}
 {% 				if loggingEnabled == True %}
 	{{schEditWire.name}}
@@
 {% endfor %}{# schEditModules #}
 {% for schEditModule in schEditModules %} {# _KiSchEditModule type #}
-{% 		for schEditConn in schEditModule.schEditConns["input"] %} {# _KiSchEditConn type #}
+{% 		for schEditConn in schEditModule.schEditConns["left"] %} {# _KiSchEditConn type #}
 {% 			for schEditNode in schEditConn.schEditNodes %} {# _KiSchEditNode type #}
 	(global_label "{{schEditNode.name}}"
-		(shape input)
+		(shape {{schEditNode.type}})
 		(at {{'%.2f' % schEditNode.x}} {{'%.2f' % schEditNode.y}} 180)
 		(fields_autoplaced yes)
@@
 {% endfor %}{# schEditModules #}
 {% for schEditModule in schEditModules %} {# _KiSchEditModule type #}
-{% 		for schEditConn in schEditModule.schEditConns["output"] %} {# _KiSchEditConn type #}
+{% 		for schEditConn in schEditModule.schEditConns["right"] %} {# _KiSchEditConn type #}
 {% 			for schEditNode in schEditConn.schEditNodes %} {# _KiSchEditNode type #}
 	(global_label "{{schEditNode.name}}"
-		(shape output)
+		(shape {{schEditNode.type}})
 		(at {{'%.2f' % schEditNode.x}} {{'%.2f' % schEditNode.y}} 0)
 		(fields_autoplaced yes)

Commit message: 19-generate-uuid-for-elements: lets make simple really simple uuid based final wires matching removing empty lines erasing random print functions from library uuids are unique validated
Parts:
- removed {{schEditModule.symEditSym.sym.designator}}1: ~, symbol {{schEditModule.libName}}:{{schEditModule.symEditSym.sym.name}}
- added {{schEditModule.symEditSym.sym.designator}}: ~, symbol {{schEditModule.libName}}:{{schEditModule.symEditSym.sym.name}}
Connections:
- net {{schEditNode.name}}: now also {{schEditModule.symEditSym.sym.designator}}.{{symEditPin.pin.number}} ({{symEditPin.pin.name}})
Changed lines of the file:
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@@
 	(generator "eeschema")
 	(generator_version "8.0")
+	(uuid "{{uuid}}")
 	(paper "User" {{pageWidth}} {{pageHeight}})
-{% for schEditModule in schEditModules %} {# _KiSchEditModule type #}
+{% for schEditModule in schEditModules %}{# _KiSchEditModule type #}
 {% 		if not schEditModule.numOfSchEditConns["left"] == 0 %}
 {% 			for schEditWire in schEditModule.schEditWireCont["left"].wires %}
@@
 			(type default)
 		)
+		(uuid "{{schEditWire.uuid}}")
 	)
 {% 			endfor %}{# schEditWire #}
-{% 		endif %} {# numOfSchEditConns #}
+{% 		endif %}{# numOfSchEditConns #}
 {% endfor %}{# schEditModules #}
-{% for schEditModule in schEditModules %} {# _KiSchEditModule type #}
+{% for schEditModule in schEditModules %}{# _KiSchEditModule type #}
 {% 		if not schEditModule.numOfSchEditConns["right"] == 0 %}
 {% 			for schEditWire in schEditModule.schEditWireCont["right"].wires %}
@@
 			(type default)
 		)
+		(uuid "{{schEditWire.uuid}}")
 	)
 {% 			endfor %}{# schEditWire #}
-{% 		endif %} {# numOfSchEditConns #}
+{% 		endif %}{# numOfSchEditConns #}
 {% endfor %}{# schEditModules #}
-{% for schEditModule in schEditModules %} {# _KiSchEditModule type #}
+{% for schEditModule in schEditModules %}{# _KiSchEditModule type #}
 {% 			for schEditWire in schEditModule.finalWires %}
 {% 				if loggingEnabled == True %}
@@
 			(type default)
 		)
+		(uuid "{{schEditWire.uuid}}")
 	)
 {% 			endfor %}{# schEditWire #}
 {% endfor %}{# schEditModules #}
-{% for schEditModule in schEditModules %} {# _KiSchEditModule type #}
-{% 		for schEditConn in schEditModule.schEditConns["left"] %} {# _KiSchEditConn type #}
-{% 			for schEditNode in schEditConn.schEditNodes %} {# _KiSchEditNode type #}
+{% for schEditModule in schEditModules %}{# _KiSchEditModule type #}
+{% 		for schEditConn in schEditModule.schEditConns["left"] %}{# _KiSchEditConn type #}
+{% 			for schEditNode in schEditConn.schEditNodes %}{# _KiSchEditNode type #}
 	(global_label "{{schEditNode.name}}"
 		(shape {{schEditNode.type}})
@@
 			(justify right)
 		)
+		(uuid "{{schEditNode.uuid}}")
 		(property "Intersheetrefs" "${INTERSHEET_REFS}"
 			(at {{'%.2f' % schEditNode.x}} {{'%.2f' % schEditNode.y}} 0)
@@
 {% 		endfor %}{# schEditConns #}
 {% endfor %}{# schEditModules #}
-{% for schEditModule in schEditModules %} {# _KiSchEditModule type #}
-{% 		for schEditConn in schEditModule.schEditConns["right"] %} {# _KiSchEditConn type #}
-{% 			for schEditNode in schEditConn.schEditNodes %} {# _KiSchEditNode type #}
+{% for schEditModule in schEditModules %}{# _KiSchEditModule type #}
+{% 		for schEditConn in schEditModule.schEditConns["right"] %}{# _KiSchEditConn type #}
+{% 			for schEditNode in schEditConn.schEditNodes %}{# _KiSchEditNode type #}
 	(global_label "{{schEditNode.name}}"
 		(shape {{schEditNode.type}})
@@
 			(justify left)
 		)
+		(uuid "{{schEditNode.uuid}}")
 		(property "Intersheetrefs" "${INTERSHEET_REFS}"
 			(at {{'%.2f' % schEditNode.x}} {{'%.2f' % schEditNode.y}} 0)
@@
 {% 		endfor %}{# schEditConns #}
 {% endfor %}{# schEditModules #}
-{% for schEditModule in schEditModules %} {# _KiSchEditModule type #}
+{% for schEditModule in schEditModules %}{# _KiSchEditModule type #}
 	(symbol
 		(lib_id "{{schEditModule.libName}}:{{schEditModule.symEditSym.sym.name}}")
@@
 		(dnp no)
 		(fields_autoplaced yes)
-		(property "Reference" "{{schEditModule.symEditSym.sym.designator}}1"
+		(uuid "{{schEditModule.uuid}}")
+		(property "Reference" "{{schEditModule.symEditSym.sym.designator}}"
 			(at {{'%.2f' % schEditModule.desigx}} {{'%.2f' % schEditModule.desigy}} 0)
 			(effects
@@
 			)
 		)
-		(pin ""
+{%		for symEditPin in schEditModule.symEditSym.symEditPins %}{# KiSymEditPin type #}
+		(pin "{{symEditPin.pin.name}}"
+			(uuid "{{symEditPin.pin.uuid}}")
 		)
+{%		endfor %}
 		(instances
 			(project ""
-				(path "/97f17985-da40-43fd-b268-8c96b481a2af"
-					(reference "{{schEditModule.symEditSym.sym.designator}}1")
+				(path "/{{uuid}}"
+					(reference "{{schEditModule.symEditSym.sym.designator}}")
 					(unit 1)
 				)

Commit message: 29-support-multiple-instantantion-of-same-symbol: single symbol in page in project modified to support multiple instantion of same symbol
Connections:
- net {{schEditNode.name}}: no longer {{schEditModule.symEditSym.sym.designator}}.{{symEditPin.pin.number}} ({{symEditPin.pin.name}})
Changed lines of the file:
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@@
 		)
 {%		for symEditPin in schEditModule.symEditSym.symEditPins %}{# KiSymEditPin type #}
+{% 			if loggingEnabled == True %}
+	{{schEditModule.symEditSym.sym.designator}}
+{% 			endif %}
 		(pin "{{symEditPin.pin.name}}"
 			(uuid "{{symEditPin.pin.uuid}}")
